File: board/ultrasonic.kicad_sch (KiCad schematic)
At the start: 21 parts, among them Q7 BSS123, Q8 BSS123, T1 B78416A2232A003, U8 PGA460TPWR

Commit message: Changed US-Transducer
Parts:
- removed LS1: Speaker, Capacitor_THT:CP_Radial_D10.0mm_P5.00mm, symbol Device:Speaker
- added LS1: HY40A16T12-1, OBSPro:HY40A16T12, symbol OBSPro:HY40A16T12-1
Connections:
- net GND: now also LS1.2
- net INP: now also LS1.1
Changed lines of the file:
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@@
-    )
-  )
-  (symbol (lib_id "Device:Speaker") (at 229.87 77.47 0) (unit 1)
-    (in_bom yes) (on_board yes) (dnp no)
-    (property "Reference" "LS1" (at 228.6 83.82 0)
-      (effects (font (size 1.27 1.27)) (justify left))
-    )
-    (property "Value" "Speaker" (at 226.06 86.36 0)
-      (effects (font (size 1.27 1.27)) (justify left))
-    )
-    (property "Footprint" "Capacitor_THT:CP_Radial_D10.0mm_P5.00mm" (at 229.87 82.55 0)
-      (effects (font (size 1.27 1.27)) hide)
-    )
-    (property "Datasheet" "~" (at 229.616 78.74 0)
-      (effects (font (size 1.27 1.27)) hide)
-    )
-    (property "Datasheet" "~" (at 229.87 77.47 0)
-      (effects (font (size 1.27 1.27)) hide)
-    )
-    (property "Reference" "LS?" (at 229.87 77.47 0)
-      (effects (font (size 1.27 1.27)) hide)
-    )
-    (property "Value" "Speaker" (at 229.87 77.47 0)
-      (effects (font (size 1.27 1.27)) hide)
-    )
-    (property "JLC_BasicPart" "no" (at 229.87 77.47 0)
-      (effects (font (size 1.27 1.27)) hide)
-    )
-    (property "JLC_PN" "C242178" (at 229.87 77.47 0)
-      (effects (font (size 1.27 1.27)) hide)
-    )
-    (property "MPN" "GU1008C-40T & GU1008C-40R" (at 229.87 77.47 0)
-      (effects (font (size 1.27 1.27)) hide)
-    )
-    (property "Manufacturer" "INGHAi" (at 229.87 77.47 0)
-      (effects (font (size 1.27 1.27)) hide)
-    )
-    (property "JLC_Price10" "1.2985" (at 229.87 77.47 0)
-      (effects (font (size 1.27 1.27)) hide)
-    )
-    (pin "1")
-    (pin "2")
-    (instances
-      (project "OBSPro"
-        (path "/1b575199-a76e-4620-8a1a-43f78ed7da24/92aed634-9154-4b6d-b7ec-aef540896df2/25fe6b58-d6b8-4d1b-be6d-69e6fb82109f"
-          (reference "LS1") (unit 1)
-        )
-        (path "/1b575199-a76e-4620-8a1a-43f78ed7da24/92aed634-9154-4b6d-b7ec-aef540896df2/4fcd8922-93f5-4d1f-8e26-f37aa513f5fd"
-          (reference "LS2") (unit 1)
-        )
-      )
     )
   )
@@
         )
       )
+    )
+  )
+  (symbol (lib_id "OBSPro:HY40A16T12-1") (at 229.87 77.47 0) (unit 1)
+    (in_bom yes) (on_board yes) (dnp no) (fields_autoplaced)
+    (property "Reference" "LS1" (at 234.95 76.2 0)
+      (effects (font (size 1.27 1.27)) (justify left))
+    )
+    (property "Value" "HY40A16T12-1" (at 234.95 78.74 0)
+      (effects (font (size 1.27 1.27)) (justify left))
+    )
+    (property "Footprint" "OBSPro:HY40A16T12" (at 229.87 82.55 0)
+      (effects (font (size 1.27 1.27)) hide)
+    )
+    (property "Datasheet" "~" (at 229.616 78.74 0)
+      (effects (font (size 1.27 1.27)) hide)
+    )
+    (property "MPN" "HY40A16T12-1" (at 229.87 77.47 0)
+      (effects (font (size 1.27 1.27)) hide)
+    )
+    (property "Manufacturer" "HYDZ" (at 234.95 81.28 0)
+      (effects (font (size 1.27 1.27)) (justify left))
+    )
+    (pin "1")
+    (pin "2")
+    (instances
+      (project "OBSPro"
+        (path "/1b575199-a76e-4620-8a1a-43f78ed7da24/92aed634-9154-4b6d-b7ec-aef540896df2/25fe6b58-d6b8-4d1b-be6d-69e6fb82109f"
+          (reference "LS1") (unit 1)
+        )
+        (path "/1b575199-a76e-4620-8a1a-43f78ed7da24/92aed634-9154-4b6d-b7ec-aef540896df2/4fcd8922-93f5-4d1f-8e26-f37aa513f5fd"
+          (reference "LS2") (unit 1)
+        )
+      )

Commit message: Updated an cleaned board with new schematic
Parts:
- LS1: JLC_BasicPart (none) -> no; JLC_PN (none) -> C17701106
Changed lines of the file:
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@@
       (effects (font (size 1.27 1.27)) (justify left))
+    )
+    (property "JLC_BasicPart" "no" (at 229.87 77.47 0)
+      (effects (font (size 1.27 1.27)) hide)
+    )
+    (property "JLC_PN" "C17701106" (at 229.87 77.47 0)
+      (effects (font (size 1.27 1.27)) hide)
     )
     (pin "1")
