File: board/sensors.kicad_sch (KiCad schematic)
At the start: 25 parts, among them J4 PROG, U6 MAX-M8C

Commit message: Everything routed, a few changes in the components, first prototypes ordered
Parts:
- added C25: 100n, Capacitor_SMD:C_0603_1608Metric, symbol Device:C_Small
- R? (x6): JLC_BasicPart (none) -> yes
- renumbered C22 to C24, C23 to C26, U6 to U7
Connections:
- net +3V3: no longer U7.7 (VCC_IO), U7.8 (VCC)
- net GND: now also C25.2; no longer AE1.2 (PCB_Trace)
- new net +3V3GPS: C25.1, U7.7 (VCC_IO), U7.8 (VCC)
- no-connect marks 8 -> 9

Commit message: Fixed ERC/DRC errors, last cleanup before production data export
Parts:
- RV1: footprint Potentiometer_THT:Potentiometer_Bourns_3266W_Vertical -> Potentiometer_SMD:Potentiometer_Bourns_TC33X_Vertical; JLC_PN C123430 -> C719174; MPN 3266W-1-103 -> TC33X-2-102E; Manufacturer BOCHEN(Chengdu Guosheng Tech) -> BOURNS
Connections:
- net +3V3: now also RV1.3; no longer RV1.1
- net GND: now also RV1.1; no longer RV1.3
Changed lines of the file:
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@@
     (pin "1")
   )
-  (symbol (lib_id "Device:R_Potentiometer_Small") (at 238.76 43.18 0) (unit 1)
+  (symbol (lib_id "Device:R_Potentiometer_Small") (at 238.76 43.18 0) (mirror x) (unit 1)
     (in_bom yes) (on_board yes)
-    (property "Reference" "RV1" (id 0) (at 243.84 40.64 0)
+    (property "Reference" "RV1" (id 0) (at 243.84 45.72 0)
       (effects (font (size 1.27 1.27)) (justify right))
     )
-    (property "Value" "1k" (id 1) (at 242.57 45.72 0)
+    (property "Value" "1k" (id 1) (at 242.57 40.64 0)
       (effects (font (size 1.27 1.27)) (justify right))
     )
-    (property "Footprint" "Potentiometer_THT:Potentiometer_Bourns_3266W_Vertical" (id 2) (at 238.76 43.18 0)
+    (property "Footprint" "Potentiometer_SMD:Potentiometer_Bourns_TC33X_Vertical" (id 2) (at 238.76 43.18 0)
       (effects (font (size 1.27 1.27)) hide)
     )
@@
       (effects (font (size 1.27 1.27)) hide)
     )
-    (property "JLC_PN" "C123430" (id 5) (at 238.76 43.18 0)
+    (property "JLC_PN" "C719174" (id 5) (at 238.76 43.18 0)
       (effects (font (size 1.27 1.27)) hide)
     )
-    (property "MPN" "3266W-1-103" (id 6) (at 238.76 43.18 0)
+    (property "MPN" "TC33X-2-102E" (id 6) (at 238.76 43.18 0)
       (effects (font (size 1.27 1.27)) hide)
     )
-    (property "Manufacturer" "BOCHEN(Chengdu Guosheng Tech)" (id 7) (at 238.76 43.18 0)
+    (property "Manufacturer" "BOURNS" (id 7) (at 238.76 43.18 0)
       (effects (font (size 1.27 1.27)) hide)
     )

Commit message: Updated price information for 10x and added a calculation for 20 boards including all parts and assembly cost
Parts:
- AE1: JLC_Price10 0.8651 -> 0.8696
- C10, C24, C25, C26: JLC_Price10 0.0042 -> 0.0021
- D4, D5: JLC_Price10 (none) -> 0.0064
- J4: JLC_Price10 (none) -> 0.0325
- R28, R29: renamed from R?; JLC_Price10 (none) -> 0.0005
- R30, R31, R32, R33, R36, R37: renamed from R?; JLC_Price10 (none) -> 0.0009
- R4, R6: JLC_Price10 (none) -> 0.0005
- RV1: JLC_Price10 (none) -> 0.1247
- U6: renamed from U?; JLC_Price10 (none) -> 0.3586
- U7: JLC_Price10 15.73 -> 15.07

Commit message: Updated schematic to new revision: Switch ultrasonic modules to PGA460, using ublox M10 GPS
Parts:
- removed C10 (x2), C24: 100n, Capacitor_SMD:C_0603_1608Metric_Pad1.08x0.95mm_HandSolder, symbol Device:C_Small
- removed J4: PROG, Connector_PinHeader_2.54mm:PinHeader_1x06_P2.54mm_Horizontal, symbol Connector_Generic:Conn_01x06
- removed R28, R29, R4 (x2), R6 (x2): 1k, Resistor_SMD:R_0603_1608Metric, symbol Device:R_Small
- removed R30, R32: 75k, Resistor_SMD:R_0603_1608Metric, symbol Device:R_Small
- removed R31, R33: R_Small, Resistor_SMD:R_0603_1608Metric, symbol Device:R_Small
- removed R36, R37: 3.3M, Resistor_SMD:R_0603_1608Metric, symbol Device:R_Small
- removed RV1: 1k, Potentiometer_SMD:Potentiometer_Bourns_TC33X_Vertical, symbol Device:R_Potentiometer_Small
- removed U6: LM393, Package_SO:SOIC-8_3.9x4.9mm_P1.27mm, symbol Comparator:LM393
- U?: renamed from U7; value MAX-M8C -> MAX-M10M; symbol RF_GPS:MAX-M8C -> OBSPro:MAX-M10M; JLC_PN (none) -> C6293820; MPN MAX-M8C-0 -> MAX-M10M-00B
Connections:
- no-connect marks 9 -> 10
Other:
- sheet Ultrasonic1 ports: added IO_3V3, MISO, MOSI, SCLK; removed COMPIN, ECHO, NRST, SIGOUT, SWIM, TRIG
- sheet Ultrasonic2 ports: added IO_3V3, MISO, MOSI, SCLK; removed COMPIN, ECHO, NRST, SIGOUT, SWIM, TRIG

Commit message: Fixed ERC errors
Parts:
- gave numbers to parts that had none: 1
- renumbered C25 to C32, C26 to C33, D4 to D5, D5 to D6
Changed lines of the file:
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@@
   (symbol (lib_id "power:GND") (at 85.09 102.87 0) (unit 1)
     (in_bom yes) (on_board yes) (dnp no) (fields_autoplaced)
-    (property "Reference" "#PWR093" (at 85.09 109.22 0)
+    (property "Reference" "#PWR094" (at 85.09 109.22 0)
       (effects (font (size 1.27 1.27)) hide)
     )
@@
       (project "OBSPro"
         (path "/1b575199-a76e-4620-8a1a-43f78ed7da24/92aed634-9154-4b6d-b7ec-aef540896df2"
-          (reference "#PWR093") (unit 1)
+          (reference "#PWR094") (unit 1)
         )
       )
@@
   (symbol (lib_id "Device:D_Small") (at 90.17 96.52 0) (unit 1)
     (in_bom yes) (on_board yes) (dnp no)
-    (property "Reference" "D4" (at 90.17 93.98 0)
+    (property "Reference" "D5" (at 90.17 93.98 0)
       (effects (font (size 1.27 1.27)))
     )
@@
       (effects (font (size 1.27 1.27)) hide)
     )
-    (pin "1")
-    (pin "2")
-    (instances
-      (project "OBSPro"
-        (path "/1b575199-a76e-4620-8a1a-43f78ed7da24/92aed634-9154-4b6d-b7ec-aef540896df2"
-          (reference "D4") (unit 1)
+    (property "Sim.Device" "D" (at 90.17 96.52 0)
+      (effects (font (size 1.27 1.27)) hide)
+    )
+    (property "Sim.Pins" "1=K 2=A" (at 90.17 96.52 0)
+      (effects (font (size 1.27 1.27)) hide)
+    )
+    (pin "1")
+    (pin "2")
+    (instances
+      (project "OBSPro"
+        (path "/1b575199-a76e-4620-8a1a-43f78ed7da24/92aed634-9154-4b6d-b7ec-aef540896df2"
+          (reference "D5") (unit 1)
         )
       )
@@
   (symbol (lib_id "power:GND") (at 31.75 100.33 0) (unit 1)
     (in_bom yes) (on_board yes) (dnp no) (fields_autoplaced)
-    (property "Reference" "#PWR091" (at 31.75 106.68 0)
+    (property "Reference" "#PWR093" (at 31.75 106.68 0)
       (effects (font (size 1.27 1.27)) hide)
     )
@@
       (project "OBSPro"
         (path "/1b575199-a76e-4620-8a1a-43f78ed7da24/92aed634-9154-4b6d-b7ec-aef540896df2"
-          (reference "#PWR091") (unit 1)
+          (reference "#PWR093") (unit 1)
         )
       )
@@
   (symbol (lib_id "OBSPro:+3V3GPS") (at 31.75 95.25 0) (unit 1)
     (in_bom yes) (on_board yes) (dnp no) (fields_autoplaced)
-    (property "Reference" "#PWR088" (at 31.75 99.06 0)
+    (property "Reference" "#PWR090" (at 31.75 99.06 0)
       (effects (font (size 1.27 1.27)) hide)
     )
@@
       (project "OBSPro"
         (path "/1b575199-a76e-4620-8a1a-43f78ed7da24/92aed634-9154-4b6d-b7ec-aef540896df2"
-          (reference "#PWR088") (unit 1)
+          (reference "#PWR090") (unit 1)
         )
       )
@@
   (symbol (lib_id "OBSPro:MAX-M10M") (at 67.31 115.57 0) (unit 1)
     (in_bom yes) (on_board yes) (dnp no) (fields_autoplaced)
-    (property "Reference" "U?" (at 69.5041 133.35 0)
+    (property "Reference" "U7" (at 69.5041 133.35 0)
       (effects (font (size 1.27 1.27)) (justify left))
     )
@@
       (project "OBSPro"
         (path "/1b575199-a76e-4620-8a1a-43f78ed7da24/92aed634-9154-4b6d-b7ec-aef540896df2"
-          (reference "U?") (unit 1)
+          (reference "U7") (unit 1)
         )
       )
@@
   (symbol (lib_id "Device:C_Small") (at 31.75 97.79 0) (unit 1)
     (in_bom yes) (on_board yes) (dnp no) (fields_autoplaced)
-    (property "Reference" "C25" (at 34.29 96.5262 0)
+    (property "Reference" "C32" (at 34.29 96.5262 0)
       (effects (font (size 1.27 1.27)) (justify left))
     )
@@
       (project "OBSPro"
         (path "/1b575199-a76e-4620-8a1a-43f78ed7da24/92aed634-9154-4b6d-b7ec-aef540896df2"
-          (reference "C25") (unit 1)
+          (reference "C32") (unit 1)
         )
       )
@@
   (symbol (lib_id "power:GND") (at 67.31 133.35 0) (unit 1)
     (in_bom yes) (on_board yes) (dnp no) (fields_autoplaced)
-    (property "Reference" "#PWR094" (at 67.31 139.7 0)
+    (property "Reference" "#PWR095" (at 67.31 139.7 0)
       (effects (font (size 1.27 1.27)) hide)
     )
@@
       (project "OBSPro"
         (path "/1b575199-a76e-4620-8a1a-43f78ed7da24/92aed634-9154-4b6d-b7ec-aef540896df2"
-          (reference "#PWR094") (unit 1)
+          (reference "#PWR095") (unit 1)
         )
       )
@@
   (symbol (lib_id "Device:C_Small") (at 85.09 100.33 0) (unit 1)
     (in_bom yes) (on_board yes) (dnp no) (fields_autoplaced)
-    (property "Reference" "C26" (at 87.63 99.0662 0)
+    (property "Reference" "C33" (at 87.63 99.0662 0)
       (effects (font (size 1.27 1.27)) (justify left))
     )
@@
       (project "OBSPro"
         (path "/1b575199-a76e-4620-8a1a-43f78ed7da24/92aed634-9154-4b6d-b7ec-aef540896df2"
-          (reference "C26") (unit 1)
+          (reference "C33") (unit 1)
         )
       )
@@
   (symbol (lib_id "Device:D_Small") (at 99.06 96.52 0) (unit 1)
     (in_bom yes) (on_board yes) (dnp no)
-    (property "Reference" "D5" (at 99.06 93.98 0)
+    (property "Reference" "D6" (at 99.06 93.98 0)
       (effects (font (size 1.27 1.27)))
     )
@@
       (effects (font (size 1.27 1.27)) hide)
     )
-    (pin "1")
-    (pin "2")
-    (instances
-      (project "OBSPro"
-        (path "/1b575199-a76e-4620-8a1a-43f78ed7da24/92aed634-9154-4b6d-b7ec-aef540896df2"
-          (reference "D5") (unit 1)
+    (property "Sim.Device" "D" (at 99.06 96.52 0)
+      (effects (font (size 1.27 1.27)) hide)
+    )
+    (property "Sim.Pins" "1=K 2=A" (at 99.06 96.52 0)
+      (effects (font (size 1.27 1.27)) hide)
+    )
+    (pin "1")
+    (pin "2")
+    (instances
+      (project "OBSPro"
+        (path "/1b575199-a76e-4620-8a1a-43f78ed7da24/92aed634-9154-4b6d-b7ec-aef540896df2"
+          (reference "D6") (unit 1)
         )
       )
@@
   (symbol (lib_id "power:+BATT") (at 105.41 95.25 0) (unit 1)
     (in_bom yes) (on_board yes) (dnp no) (fields_autoplaced)
-    (property "Reference" "#PWR090" (at 105.41 99.06 0)
+    (property "Reference" "#PWR092" (at 105.41 99.06 0)
       (effects (font (size 1.27 1.27)) hide)
     )
@@
       (project "OBSPro"
         (path "/1b575199-a76e-4620-8a1a-43f78ed7da24/92aed634-9154-4b6d-b7ec-aef540896df2"
-          (reference "#PWR090") (unit 1)
+          (reference "#PWR092") (unit 1)
         )
       )
@@
   (symbol (lib_id "OBSPro:+3V3GPS") (at 62.23 95.25 0) (unit 1)
     (in_bom yes) (on_board yes) (dnp no) (fields_autoplaced)
-    (property "Reference" "#PWR089" (at 62.23 99.06 0)
+    (property "Reference" "#PWR091" (at 62.23 99.06 0)
       (effects (font (size 1.27 1.27)) hide)
     )
@@
       (project "OBSPro"
         (path "/1b575199-a76e-4620-8a1a-43f78ed7da24/92aed634-9154-4b6d-b7ec-aef540896df2"
-          (reference "#PWR089") (unit 1)
+          (reference "#PWR091") (unit 1)
         )
       )
@@
   (symbol (lib_id "power:PWR_FLAG") (at 80.01 95.25 0) (unit 1)
     (in_bom yes) (on_board yes) (dnp no)
-    (property "Reference" "#FLG05" (at 80.01 93.345 0)
+    (property "Reference" "#FLG06" (at 80.01 93.345 0)
       (effects (font (size 1.27 1.27)) hide)
     )
@@
       (project "OBSPro"
         (path "/1b575199-a76e-4620-8a1a-43f78ed7da24/92aed634-9154-4b6d-b7ec-aef540896df2"
-          (reference "#FLG05") (unit 1)
-        )
-      )
+          (reference "#FLG06") (unit 1)
+        )
+      )

Commit message: Rough placement of US electronics
Parts:
- renumbered D5 to D4, D6 to D5
Changed lines of the file:
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@@
   (symbol (lib_id "power:GND") (at 85.09 102.87 0) (unit 1)
     (in_bom yes) (on_board yes) (dnp no) (fields_autoplaced)
-    (property "Reference" "#PWR094" (at 85.09 109.22 0)
+    (property "Reference" "#PWR092" (at 85.09 109.22 0)
       (effects (font (size 1.27 1.27)) hide)
     )
@@
       (project "OBSPro"
         (path "/1b575199-a76e-4620-8a1a-43f78ed7da24/92aed634-9154-4b6d-b7ec-aef540896df2"
-          (reference "#PWR094") (unit 1)
+          (reference "#PWR092") (unit 1)
         )
       )
@@
   (symbol (lib_id "Device:D_Small") (at 90.17 96.52 0) (unit 1)
     (in_bom yes) (on_board yes) (dnp no)
-    (property "Reference" "D5" (at 90.17 93.98 0)
+    (property "Reference" "D4" (at 90.17 93.98 0)
       (effects (font (size 1.27 1.27)))
     )
@@
       (project "OBSPro"
         (path "/1b575199-a76e-4620-8a1a-43f78ed7da24/92aed634-9154-4b6d-b7ec-aef540896df2"
-          (reference "D5") (unit 1)
+          (reference "D4") (unit 1)
         )
       )
@@
   (symbol (lib_id "power:GND") (at 31.75 100.33 0) (unit 1)
     (in_bom yes) (on_board yes) (dnp no) (fields_autoplaced)
-    (property "Reference" "#PWR093" (at 31.75 106.68 0)
+    (property "Reference" "#PWR091" (at 31.75 106.68 0)
       (effects (font (size 1.27 1.27)) hide)
     )
@@
       (project "OBSPro"
         (path "/1b575199-a76e-4620-8a1a-43f78ed7da24/92aed634-9154-4b6d-b7ec-aef540896df2"
-          (reference "#PWR093") (unit 1)
+          (reference "#PWR091") (unit 1)
         )
       )
@@
   (symbol (lib_id "OBSPro:+3V3GPS") (at 31.75 95.25 0) (unit 1)
     (in_bom yes) (on_board yes) (dnp no) (fields_autoplaced)
-    (property "Reference" "#PWR090" (at 31.75 99.06 0)
+    (property "Reference" "#PWR088" (at 31.75 99.06 0)
       (effects (font (size 1.27 1.27)) hide)
     )
@@
       (project "OBSPro"
         (path "/1b575199-a76e-4620-8a1a-43f78ed7da24/92aed634-9154-4b6d-b7ec-aef540896df2"
-          (reference "#PWR090") (unit 1)
+          (reference "#PWR088") (unit 1)
         )
       )
@@
   (symbol (lib_id "power:GND") (at 67.31 133.35 0) (unit 1)
     (in_bom yes) (on_board yes) (dnp no) (fields_autoplaced)
-    (property "Reference" "#PWR095" (at 67.31 139.7 0)
+    (property "Reference" "#PWR093" (at 67.31 139.7 0)
       (effects (font (size 1.27 1.27)) hide)
     )
@@
       (project "OBSPro"
         (path "/1b575199-a76e-4620-8a1a-43f78ed7da24/92aed634-9154-4b6d-b7ec-aef540896df2"
-          (reference "#PWR095") (unit 1)
+          (reference "#PWR093") (unit 1)
         )
       )
@@
   (symbol (lib_id "Device:D_Small") (at 99.06 96.52 0) (unit 1)
     (in_bom yes) (on_board yes) (dnp no)
-    (property "Reference" "D6" (at 99.06 93.98 0)
+    (property "Reference" "D5" (at 99.06 93.98 0)
       (effects (font (size 1.27 1.27)))
     )
@@
       (project "OBSPro"
         (path "/1b575199-a76e-4620-8a1a-43f78ed7da24/92aed634-9154-4b6d-b7ec-aef540896df2"
-          (reference "D6") (unit 1)
+          (reference "D5") (unit 1)
         )
       )
@@
   (symbol (lib_id "power:+BATT") (at 105.41 95.25 0) (unit 1)
     (in_bom yes) (on_board yes) (dnp no) (fields_autoplaced)
-    (property "Reference" "#PWR092" (at 105.41 99.06 0)
+    (property "Reference" "#PWR090" (at 105.41 99.06 0)
       (effects (font (size 1.27 1.27)) hide)
     )
@@
       (project "OBSPro"
         (path "/1b575199-a76e-4620-8a1a-43f78ed7da24/92aed634-9154-4b6d-b7ec-aef540896df2"
-          (reference "#PWR092") (unit 1)
+          (reference "#PWR090") (unit 1)
         )
       )
@@
   (symbol (lib_id "OBSPro:+3V3GPS") (at 62.23 95.25 0) (unit 1)
     (in_bom yes) (on_board yes) (dnp no) (fields_autoplaced)
-    (property "Reference" "#PWR091" (at 62.23 99.06 0)
+    (property "Reference" "#PWR089" (at 62.23 99.06 0)
       (effects (font (size 1.27 1.27)) hide)
     )
@@
       (project "OBSPro"
         (path "/1b575199-a76e-4620-8a1a-43f78ed7da24/92aed634-9154-4b6d-b7ec-aef540896df2"
-          (reference "#PWR091") (unit 1)
-        )
-      )
+          (reference "#PWR089") (unit 1)
+        )
+      )

Commit message: 3D-Modelle hinzugefügt
Parts:
- U7: footprint RF_GPS:ublox_MAX -> OBSPro:ublox_MAX
Changed lines of the file:
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@@
       (effects (font (size 1.27 1.27)) (justify left))
     )
-    (property "Footprint" "RF_GPS:ublox_MAX" (at 77.47 132.08 0)
+    (property "Footprint" "OBSPro:ublox_MAX" (at 77.47 132.08 0)
       (effects (font (size 1.27 1.27)) hide)
     )
@@
       (effects (font (size 1.27 1.27)) hide)
     )
+    (property "MF" "" (at 67.31 115.57 0)
+      (effects (font (size 1.27 1.27)) hide)
+    )
+    (property "Farnell_PN" "" (at 67.31 115.57 0)
+      (effects (font (size 1.27 1.27)) hide)
+    )
+    (property "Mouser_PN" "" (at 67.31 115.57 0)
+      (effects (font (size 1.27 1.27)) hide)
+    )
